File: mainboard/_autosave-mainboard.sch (KiCad schematic (older format))
At the start: 107 parts, among them J1 USB_B_Micro, J2 Conn_01x19_MountingPin, J3 Conn_01x19_MountingPin, J4 Conn_01x02_Male, Q1 DMG2301L, Q2 MMBT3904, Q3 MMBT3904, SW1 SW_Push, SW2 SW_Push, U1 ESP32-WROOM-32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

Commit message: More WIP
Connections:
- net +3V3: now also D6.2 (A), U6.5 (SDO); no longer R26.1
- net GND: now also R23.2, R24.2, R25.2, R26.2, R27.2, R28.2, R29.2; no longer D3.1 (K), D4.1 (K), D5.1 (K), D6.1 (K), D7.1 (K), D8.1 (K), D9.1 (K), U6.5 (SDO)
- net IO4: now also D9.2 (A); no longer R29.1
- net VBUS: now also D5.2 (A); no longer R25.1
- net VCC_EAR0: now also D7.2 (A); no longer R27.1
- net VCC_EAR1: now also D8.2 (A); no longer R28.1
- net VDC: now also D3.2 (A); no longer R23.1
- net VUSB: now also D4.2 (A); no longer R24.1
- new net: D3.1 (K), R23.1
- new net: D4.1 (K), R24.1
- new net: D5.1 (K), R25.1
- new net: D6.1 (K), R26.1
- new net: D7.1 (K), R27.1
- new net: D8.1 (K), R28.1
- new net: D9.1 (K), R29.1
Other:
- moved on the sheet: D3, D4, D5, D6, D7, D8, D9, R23, R24, R25, R26, R27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
Changed lines of the file:
@@
 	9200 10100 9200 9100
 Wire Wire Line
-	9200 9100 8200 9100
+	9200 9100 8800 9100
 Wire Wire Line
 	7250 10550 8000 10550
@@
 L Device:R R23
 U 1 1 5E46A879
+P 16300 4850
+F 0 "R23" H 16370 4896 50  0000 L CNN
+F 1 "1 kR" H 16370 4805 50  0000 L CNN
+F 2 "Resistor_SMD:R_0805_2012Metric" V 16230 4850 50  0001 C CNN
+F 3 "~" H 16300 4850 50  0001 C CNN
+	1    16300 4850
+	1    0    0    -1
+$EndComp
+$Comp
+L Device:LED D3
+U 1 1 5E46B8C6
 P 16300 4500
-F 0 "R23" H 16370 4546 50  0000 L CNN
-F 1 "1 kR" H 16370 4455 50  0000 L CNN
-F 2 "Resistor_SMD:R_0805_2012Metric" V 16230 4500 50  0001 C CNN
+F 0 "D3" V 16339 4383 50  0000 R CNN
+F 1 "LED" V 16248 4383 50  0000 R CNN
+F 2 "LED_SMD:LED_0805_2012Metric" H 16300 4500 50  0001 C CNN
 F 3 "~" H 16300 4500 50  0001 C CNN
 	1    16300 4500
-	1    0    0    -1
-$EndComp
-$Comp
-L Device:LED D3
-U 1 1 5E46B8C6
-P 16300 4850
-F 0 "D3" V 16339 4733 50  0000 R CNN
-F 1 "LED" V 16248 4733 50  0000 R CNN
-F 2 "LED_SMD:LED_0805_2012Metric" H 16300 4850 50  0001 C CNN
-F 3 "~" H 16300 4850 50  0001 C CNN
-	1    16300 4850
 	0    -1   -1   0
 $EndComp
@@
 L Device:R R24
 U 1 1 5E59D4D8
-P 16800 4500
-F 0 "R24" H 16870 4546 50  0000 L CNN
-F 1 "330 R" H 16870 4455 50  0000 L CNN
-F 2 "Resistor_SMD:R_0805_2012Metric" V 16730 4500 50  0001 C CNN
-F 3 "~" H 16800 4500 50  0001 C CNN
-	1    16800 4500
+P 16800 4850
+F 0 "R24" H 16870 4896 50  0000 L CNN
+F 1 "330 R" H 16870 4805 50  0000 L CNN
+F 2 "Resistor_SMD:R_0805_2012Metric" V 16730 4850 50  0001 C CNN
+F 3 "~" H 16800 4850 50  0001 C CNN
+	1    16800 4850
 	1    0    0    -1
 $EndComp
@@
 L Device:R R25
 U 1 1 5E59E276
-P 17300 4500
-F 0 "R25" H 17370 4546 50  0000 L CNN
-F 1 "1 kR" H 17370 4455 50  0000 L CNN
-F 2 "Resistor_SMD:R_0805_2012Metric" V 17230 4500 50  0001 C CNN
-F 3 "~" H 17300 4500 50  0001 C CNN
-	1    17300 4500
+P 17300 4850
+F 0 "R25" H 17370 4896 50  0000 L CNN
+F 1 "1 kR" H 17370 4805 50  0000 L CNN
+F 2 "Resistor_SMD:R_0805_2012Metric" V 17230 4850 50  0001 C CNN
+F 3 "~" H 17300 4850 50  0001 C CNN
+	1    17300 4850
 	1    0    0    -1
 $EndComp
@@
 L Device:R R26
 U 1 1 5E5A0416
+P 17800 4850
+F 0 "R26" H 17870 4896 50  0000 L CNN
+F 1 "220 R" H 17870 4805 50  0000 L CNN
+F 2 "Resistor_SMD:R_0805_2012Metric" V 17730 4850 50  0001 C CNN
+F 3 "~" H 17800 4850 50  0001 C CNN
+	1    17800 4850
+	1    0    0    -1
+$EndComp
+$Comp
+L Device:LED D4
+U 1 1 5E5A127C
+P 16800 4500
+F 0 "D4" V 16839 4383 50  0000 R CNN
+F 1 "LED" V 16748 4383 50  0000 R CNN
+F 2 "LED_SMD:LED_0805_2012Metric" H 16800 4500 50  0001 C CNN
+F 3 "~" H 16800 4500 50  0001 C CNN
+	1    16800 4500
+	0    -1   -1   0
+$EndComp
+$Comp
+L Device:LED D5
+U 1 1 5E5A26C1
+P 17300 4500
+F 0 "D5" V 17339 4383 50  0000 R CNN
+F 1 "LED" V 17248 4383 50  0000 R CNN
+F 2 "LED_SMD:LED_0805_2012Metric" H 17300 4500 50  0001 C CNN
+F 3 "~" H 17300 4500 50  0001 C CNN
+	1    17300 4500
+	0    -1   -1   0
+$EndComp
+$Comp
+L Device:LED D6
+U 1 1 5E5A377A
 P 17800 4500
-F 0 "R26" H 17870 4546 50  0000 L CNN
-F 1 "220 R" H 17870 4455 50  0000 L CNN
-F 2 "Resistor_SMD:R_0805_2012Metric" V 17730 4500 50  0001 C CNN
+F 0 "D6" V 17839 4383 50  0000 R CNN
+F 1 "LED" V 17748 4383 50  0000 R CNN
+F 2 "LED_SMD:LED_0805_2012Metric" H 17800 4500 50  0001 C CNN
 F 3 "~" H 17800 4500 50  0001 C CNN
 	1    17800 4500
-	1    0    0    -1
-$EndComp
-$Comp
-L Device:LED D4
-U 1 1 5E5A127C
-P 16800 4850
-F 0 "D4" V 16839 4733 50  0000 R CNN
-F 1 "LED" V 16748 4733 50  0000 R CNN
-F 2 "LED_SMD:LED_0805_2012Metric" H 16800 4850 50  0001 C CNN
-F 3 "~" H 16800 4850 50  0001 C CNN
-	1    16800 4850
-	0    -1   -1   0
-$EndComp
-$Comp
-L Device:LED D5
-U 1 1 5E5A26C1
-P 17300 4850
-F 0 "D5" V 17339 4733 50  0000 R CNN
-F 1 "LED" V 17248 4733 50  0000 R CNN
-F 2 "LED_SMD:LED_0805_2012Metric" H 17300 4850 50  0001 C CNN
-F 3 "~" H 17300 4850 50  0001 C CNN
-	1    17300 4850
-	0    -1   -1   0
-$EndComp
-$Comp
-L Device:LED D6
-U 1 1 5E5A377A
-P 17800 4850
-F 0 "D6" V 17839 4733 50  0000 R CNN
-F 1 "LED" V 17748 4733 50  0000 R CNN
-F 2 "LED_SMD:LED_0805_2012Metric" H 17800 4850 50  0001 C CNN
-F 3 "~" H 17800 4850 50  0001 C CNN
-	1    17800 4850
 	0    -1   -1   0
 $EndComp
@@
 L Device:R R27
 U 1 1 5E8A4DD7
+P 18550 4850
+F 0 "R27" H 18620 4896 50  0000 L CNN
+F 1 "470 R" H 18620 4805 50  0000 L CNN
+F 2 "Resistor_SMD:R_0805_2012Metric" V 18480 4850 50  0001 C CNN
+F 3 "~" H 18550 4850 50  0001 C CNN
+	1    18550 4850
+	1    0    0    -1
+$EndComp
+Wire Wire Line
+	18550 4350 18550 4050
+Wire Wire Line
+	18550 4050 18450 4050
+$Comp
+L Device:LED D7
+U 1 1 5E8F3B82
 P 18550 4500
-F 0 "R27" H 18620 4546 50  0000 L CNN
-F 1 "470 R" H 18620 4455 50  0000 L CNN
-F 2 "Resistor_SMD:R_0805_2012Metric" V 18480 4500 50  0001 C CNN
+F 0 "D7" V 18589 4383 50  0000 R CNN
+F 1 "LED" V 18498 4383 50  0000 R CNN
+F 2 "LED_SMD:LED_0805_2012Metric" H 18550 4500 50  0001 C CNN
 F 3 "~" H 18550 4500 50  0001 C CNN
 	1    18550 4500
-	1    0    0    -1
-$EndComp
-Wire Wire Line
-	18550 4350 18550 4050
-Wire Wire Line
-	18550 4050 18450 4050
-$Comp
-L Device:LED D7
-U 1 1 5E8F3B82
-P 18550 4850
-F 0 "D7" V 18589 4733 50  0000 R CNN
-F 1 "LED" V 18498 4733 50  0000 R CNN
-F 2 "LED_SMD:LED_0805_2012Metric" H 18550 4850 50  0001 C CNN
-F 3 "~" H 18550 4850 50  0001 C CNN
-	1    18550 4850
 	0    -1   -1   0
 $EndComp
@@
 L Device:R R28
 U 1 1 5E9DF78E
+P 19250 4850
+F 0 "R28" H 19320 4896 50  0000 L CNN
+F 1 "470 R" H 19320 4805 50  0000 L CNN
+F 2 "Resistor_SMD:R_0805_2012Metric" V 19180 4850 50  0001 C CNN
+F 3 "~" H 19250 4850 50  0001 C CNN
+	1    19250 4850
+	1    0    0    -1
+$EndComp
+Wire Wire Line
+	19250 4350 19250 4050
+Wire Wire Line
+	19250 4050 19150 4050
+$Comp
+L Device:LED D8
+U 1 1 5E9DF796
 P 19250 4500
-F 0 "R28" H 19320 4546 50  0000 L CNN
-F 1 "470 R" H 19320 4455 50  0000 L CNN
-F 2 "Resistor_SMD:R_0805_2012Metric" V 19180 4500 50  0001 C CNN
+F 0 "D8" V 19289 4383 50  0000 R CNN
+F 1 "LED" V 19198 4383 50  0000 R CNN
+F 2 "LED_SMD:LED_0805_2012Metric" H 19250 4500 50  0001 C CNN
 F 3 "~" H 19250 4500 50  0001 C CNN
 	1    19250 4500
-	1    0    0    -1
-$EndComp
-Wire Wire Line
-	19250 4350 19250 4050
-Wire Wire Line
-	19250 4050 19150 4050
-$Comp
-L Device:LED D8
-U 1 1 5E9DF796
-P 19250 4850
-F 0 "D8" V 19289 4733 50  0000 R CNN
-F 1 "LED" V 19198 4733 50  0000 R CNN
-F 2 "LED_SMD:LED_0805_2012Metric" H 19250 4850 50  0001 C CNN
-F 3 "~" H 19250 4850 50  0001 C CNN
-	1    19250 4850
 	0    -1   -1   0
 $EndComp
@@
 L Device:R R29
 U 1 1 5EA7E785
+P 19750 4850
+F 0 "R29" H 19820 4896 50  0000 L CNN
+F 1 "220 R" H 19820 4805 50  0000 L CNN
+F 2 "Resistor_SMD:R_0805_2012Metric" V 19680 4850 50  0001 C CNN
+F 3 "~" H 19750 4850 50  0001 C CNN
+	1    19750 4850
+	1    0    0    -1
+$EndComp
+$Comp
+L Device:LED D9
+U 1 1 5EA7F747
 P 19750 4500
-F 0 "R29" H 19820 4546 50  0000 L CNN
-F 1 "220 R" H 19820 4455 50  0000 L CNN
-F 2 "Resistor_SMD:R_0805_2012Metric" V 19680 4500 50  0001 C CNN
+F 0 "D9" V 19789 4383 50  0000 R CNN
+F 1 "LED" V 19698 4383 50  0000 R CNN
+F 2 "LED_SMD:LED_0805_2012Metric" H 19750 4500 50  0001 C CNN
 F 3 "~" H 19750 4500 50  0001 C CNN
 	1    19750 4500
-	1    0    0    -1
-$EndComp
-$Comp
-L Device:LED D9
-U 1 1 5EA7F747
-P 19750 4850
-F 0 "D9" V 19789 4733 50  0000 R CNN
-F 1 "LED" V 19698 4733 50  0000 R CNN
-F 2 "LED_SMD:LED_0805_2012Metric" H 19750 4850 50  0001 C CNN
-F 3 "~" H 19750 4850 50  0001 C CNN
-	1    19750 4850
 	0    -1   -1   0
 $EndComp
@@
 	8700 9500 8800 9500
 Wire Wire Line
-	8800 9500 8800 10550
-Wire Wire Line
-	8800 10550 8200 10550
-Connection ~ 8200 10550
-Wire Wire Line
 	7550 12400 7450 12400
 Wire Wire Line
@@
 Wire Wire Line
 	9700 11750 9150 11750
+Connection ~ 9150 11750
+Wire Wire Line
+	8800 9500 8800 9100
 Wire Bus Line
 	8350 2150 8350 2500
 Wire Bus Line
 	9350 2500 9350 2750
-Connection ~ 9150 11750
+Connection ~ 8800 9100
+Wire Wire Line
+	8800 9100 8200 9100
 $EndSCHEMATC
